File: hardware/boards/backplane/backplane_slot_connectors.kicad_sch (KiCad schematic)
At the start: 18 parts, among them J2 SLOT_1, J3 SLOT_2, J4 SLOT_3, J5 SLOT_4, J6 SLOT_5, J7 SLOT_6

Commit message: add ESD protection to `SLOT_1`
Parts:
- added D8: LOW_CAP_TVS, Diode_SMD:D_SOD-523, symbol Device:D_TVS
- added R3: 47R, Resistor_SMD:R_0603_1608Metric, symbol Device:R
- renumbered D9 to D10, D15 to D11, D17 to D12, D11 to D13, D13 to D7, D7 to D9, J5 to J2, J2 to J3, J3 to J4, J6 to J5, J7 to J6, J4 to J7, R8 to R2, R2 to R4, R4 to R5, R10 to R6, R12 to R7, R6 to R8
Connections:
- net GND: now also D8.2 (A2)
- net SCL_SLOT_1_CONN: now also R3.1; no longer J3.3 (Pin_3)
- new net: D8.1 (A1), J3.3 (Pin_3), R3.2
Other:
- moved on the sheet: D10, D11, D12, D13, D9, J3, J4, J5, J6, J7, R4, R5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
