File: hardware/boards/backplane/backplane_i2c_mux.kicad_sch (KiCad schematic)
At the start: 7 parts, among them J1 SPARE_I2C, U1 TCA9548APWR

Commit message: Assign vertical pin header footprint to J1
Parts:
- J1: footprint (none) -> Connector_PinHeader_2.54mm:PinHeader_1x04_P2.54mm_Vertical
Changed lines of the file:
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@@
 			)
 		)
-		(property "Footprint" ""
+		(property "Footprint" "Connector_PinHeader_2.54mm:PinHeader_1x04_P2.54mm_Vertical"
 			(at 167.64 59.69 0)
 			(hide yes)
