File: hardware/boards/backplane/05_buck_converters.kicad_sch (KiCad schematic)
At the start: 29 parts, among them U2 LM5164DDAR, U3 LM5164DDAR

Commit message: Retune backplane 12V buck ripple injection with shared BOM parts
Parts:
- added R25, R26: 110k 1%, Resistor_SMD:R_0603_1608Metric, symbol Device:R
- C12: value 3.3nF 50V X7R -> 2.2nF 50V; LCSC C92203 -> C1604; MPN 0603B332K500NT -> 0603B222K500NT
- R9: value 453k 1% -> 110k 1%; LCSC C25818 -> C25805; MPN 0603WAF4533T5E -> 0603WAF1103T5E
Connections:
- net SW_12V: now also R26.1; no longer R9.1
- new net: R25.1, R26.2
- new net: R25.2, R9.1
Other:
- note added: "NOTES: - Both regulators are LM5164DDAR at approximately 300 kHz with 100 µH inductors. - The +12 V Type-3 network is retuned for 21.6-55 V at U3 VIN (24-50 V nominal, +/-10%). - R9 + R25 + R26 = 330 kohm; C12 = 2.2 nF; C13 = 56 pF. Reuses existing BOM parts. - Verify FB injection, +12 V accuracy and load transients across input voltage and temperature. - +3V3 reuses carrier's schematic. - Input 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"
- note removed: "NOTES: - Both regulators are LM5164DDAR at approximately 300 kHz with 100 µH inductors. - The +12 V rail follows TI's 12 V / 1 A Type-3 network except for the qualified 100 µH inductor. - +3V3 reuses carrier's schematic. - Input ceramics are rated for 100 V. - Each rail uses two 22 µF / 25 V output capacitors. TODO: - [ ] Verify VIN ringing at each regulator, output ripple, PGOOD inductor tempera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"

Commit message: docs(hardware): clarify carrier voltage limits and qualification TODOs
Other:
- note added: "NOTES: - Both regulators are LM5164DDAR at approximately 300 kHz with 100 µH inductors. - The +12 V Type-3 network is retuned for 21.6-55 V at U3 VIN (qualification corners; system is 24-48 V nominal). - R9 + R25 + R26 = 330 kohm; C12 = 2.2 nF; C13 = 56 pF. Reuses existing BOM parts. - Verify FB injection, +12 V accuracy and load transients across input voltage and temperature. - +3V3 reuses carr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"
- note removed: "NOTES: - Both regulators are LM5164DDAR at approximately 300 kHz with 100 µH inductors. - The +12 V Type-3 network is retuned for 21.6-55 V at U3 VIN (24-50 V nominal, +/-10%). - R9 + R25 + R26 = 330 kohm; C12 = 2.2 nF; C13 = 56 pF. Reuses existing BOM parts. - Verify FB injection, +12 V accuracy and load transients across input voltage and temperature. - +3V3 reuses carrier's schematic. - Input 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"
Changed lines of the file:
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@@
 		)
 	)
-	(text "NOTES:\n\n  - Both regulators are LM5164DDAR at approximately 300 kHz with 100 µH inductors.\n  - The +12 V Type-3 network is retuned for 21.6-55 V at U3 VIN (24-50 V nominal, +/-10%).\n  - R9 + R25 + R26 = 330 kohm; C12 = 2.2 nF; C13 = 56 pF. Reuses existing BOM parts.\n  - Verify FB injection, +12 V accuracy and load transients across input voltage and temperature.\n  - +3V3 reuses carrier's schematic.\n  - Input ceramics are rated for 100 V.\n  - Each rail uses two 22 µF / 25 V output capacitors.\n\nTODO:\n\n  - [ ] Verify VIN ringing at each regulator, output ripple, PGOOD inductor temperature, and fan startup/stall.\n\nLAYOUT:\n\n  - Place input ceramics directly at each regulator's VIN/GND pins with a minimum-area loop.\n  - Place L1/L2 close to SW and minimize the SW copper area.\n  - Place C4/C14 at L1's output and C10/C11 at L2's output; return each pair directly to regulator GND/EP.\n  - Keep feedback and ripple-injection parts close to FB and away from SW."
+	(text "NOTES:\n\n  - Both regulators are LM5164DDAR at approximately 300 kHz with 100 µH inductors.\n  - The +12 V Type-3 network is retuned for 21.6-55 V at U3 VIN (qualification corners; system is 24-48 V nominal).\n  - R9 + R25 + R26 = 330 kohm; C12 = 2.2 nF; C13 = 56 pF. Reuses existing BOM parts.\n  - Verify FB injection, +12 V accuracy and load transients across input voltage and temperature.\n  - +3V3 reuses carrier's schematic.\n  - Input ceramics are rated for 100 V.\n  - Each rail uses two 22 µF / 25 V output capacitors.\n\nTODO:\n\n  - [ ] Verify VIN ringing at each regulator, output ripple, PGOOD, and fan startup/stall.\n  - [ ] Verify effective C1/C2/C7/C8 input and C4/C10/C11/C14 output capacitance with DC bias, tolerance and temperature.\n  - [ ] Measure U2/U3, L1/L2 and capacitor temperatures at worst load, input, ambient and enclosure airflow.\n\nLAYOUT:\n\n  - Place input ceramics directly at each regulator's VIN/GND pins with a minimum-area loop.\n  - Place L1/L2 close to SW and minimize the SW copper area.\n  - Place C4/C14 at L1's output and C10/C11 at L2's output; return each pair directly to regulator GND/EP.\n  - Keep feedback and ripple-injection parts close to FB and away from SW."
 		(exclude_from_sim no)
-		(at 14.986 55.88 0)
+		(at 14.986 59.944 0)
 		(effects
 			(font

Commit message: Use JLCPCB Basic 330k resistor for 12V ripple injection
Parts:
- removed R25, R26: 110k 1%, Resistor_SMD:R_0603_1608Metric, symbol Device:R
- R9: value 110k 1% -> 330k 1%; LCSC C25805 -> C23137; MPN 0603WAF1103T5E -> 0603WAF3303T5E
Connections:
- net SW_12V: now also R9.1
Other:
- note added: "NOTES: - Both regulators are LM5164DDAR at approximately 300 kHz with 100 µH inductors. - The +12 V Type-3 network is retuned for 21.6-55 V at U3 VIN (qualification corners; system is 24-48 V nominal). - R9 = 330 kohm (C23137, JLCPCB Basic); C12 = 2.2 nF; C13 = 56 pF. - Verify FB injection, +12 V accuracy and load transients across input voltage and temperature. - +3V3 reuses carrier's schematic.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"
- note removed: "NOTES: - Both regulators are LM5164DDAR at approximately 300 kHz with 100 µH inductors. - The +12 V Type-3 network is retuned for 21.6-55 V at U3 VIN (qualification corners; system is 24-48 V nominal). - R9 + R25 + R26 = 330 kohm; C12 = 2.2 nF; C13 = 56 pF. Reuses existing BOM parts. - Verify FB injection, +12 V accuracy and load transients across input voltage and temperature. - +3V3 reuses carr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"
