File: hardware/boards/backplane-backpack/backplane-prototype-mate.kicad_sch (KiCad schematic)
At the start: 0 parts

Commit message: hardware: add CAN-I2C gateway schematic
Other:
- added sheet CAN Fan and Status (04_can_fan_led.kicad_sch)
- added sheet I2C Multiplexer and Ports (03_i2c.kicad_sch)
- added sheet MCU and Debug (02_controller.kicad_sch)
- added sheet Power Entry and Regulators (01_power.kicad_sch)
- note added: "CAN ↔ I2C GATEWAY — REV A"
- note added: "Canonical rails: VIN_RAW (~20–36 V) → +3V3 and +12V_FAN using two LMR51610 buck converters."
- note added: "Design source: _llm/can_i2c_gateway_handoff.md and can_i2c_gateway_bom.csv"
- note added: "Four functional pages keep power conversion, MCU/debug, repeated I2C ports, and external interfaces reviewable."
- note added: "Population notes: R3–R14 DNP by default; D2/C20 DNP pending source limits; SJ1 open; SJ2/SJ3 configure fan mode."
- title: (none) -> CAN ↔ I2C Gateway
Changed lines of the file:
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@@
 (kicad_sch (version 20250114) (generator "KiCAD-MCP-Server")
   (paper "A4")
-  (sheet_instances
+  (title_block
+    (title "CAN ↔ I2C Gateway")
+    (rev "A")
+  )
+    (sheet (at 30.0 35.0) (size 75.0 45.0) (fields_autoplaced yes)
+    (stroke (width 0.0006) (type default))
+    (fill (color 0 0 0 0.0000))
+    (property "Sheet name" "Power Entry and Regulators" (at 32.54 33.73 0)
+      (effects (font (size 1.27 1.27)) (justify left bottom))
+    )
+    (property "Sheet file" "01_power.kicad_sch" (at 32.54 81.27 0)
+      (effects (font (size 1.27 1.27)) (justify left bottom))
+    )
+  )
+    (sheet (at 120.0 35.0) (size 75.0 45.0) (fields_autoplaced yes)
+    (stroke (width 0.0006) (type default))
+    (fill (color 0 0 0 0.0000))
+    (property "Sheet name" "MCU and Debug" (at 122.54 33.73 0)
+      (effects (font (size 1.27 1.27)) (justify left bottom))
+    )
+    (property "Sheet file" "02_controller.kicad_sch" (at 122.54 81.27 0)
+      (effects (font (size 1.27 1.27)) (justify left bottom))
+    )
+  )
+    (sheet (at 30.0 105.0) (size 75.0 45.0) (fields_autoplaced yes)
+    (stroke (width 0.0006) (type default))
+    (fill (color 0 0 0 0.0000))
+    (property "Sheet name" "I2C Multiplexer and Ports" (at 32.54 103.73 0)
+      (effects (font (size 1.27 1.27)) (justify left bottom))
+    )
+    (property "Sheet file" "03_i2c.kicad_sch" (at 32.54 151.27 0)
+      (effects (font (size 1.27 1.27)) (justify left bottom))
+    )
+  )
+    (sheet (at 120.0 105.0) (size 75.0 45.0) (fields_autoplaced yes)
+    (stroke (width 0.0006) (type default))
+    (fill (color 0 0 0 0.0000))
+    (property "Sheet name" "CAN Fan and Status" (at 122.54 103.73 0)
+      (effects (font (size 1.27 1.27)) (justify left bottom))
+    )
+    (property "Sheet file" "04_can_fan_led.kicad_sch" (at 122.54 151.27 0)
+      (effects (font (size 1.27 1.27)) (justify left bottom))
+    )
+  )
+	(text "CAN ↔ I2C GATEWAY — REV A"
+		(exclude_from_sim no)
+		(at 25.4 17.78 0)
+		(effects
+			(font
+				(size 2.2 2.2)
+				(bold yes)
+			)
+			(justify left bottom)
+		)
+	)
+	(text "Canonical rails: VIN_RAW (~20–36 V) → +3V3 and +12V_FAN using two LMR51610 buck converters."
+		(exclude_from_sim no)
+		(at 25.4 25.4 0)
+		(effects
+			(font
+				(size 1.2 1.2)
+			)
+			(justify left bottom)
+		)
+	)
+	(text "Four functional pages keep power conversion, MCU/debug, repeated I2C ports, and external interfaces reviewable."
+		(exclude_from_sim no)
+		(at 25.4 30.48 0)
+		(effects
+			(font
+				(size 1.1 1.1)
+			)
+			(justify left bottom)
+		)
+	)
+	(text "Population notes: R3–R14 DNP by default; D2/C20 DNP pending source limits; SJ1 open; SJ2/SJ3 configure fan mode."
+		(exclude_from_sim no)
+		(at 25.4 170.18 0)
+		(effects
+			(font
+				(size 1.1 1.1)
+			)
+			(justify left bottom)
+		)
+	)
+	(text "Design source: _llm/can_i2c_gateway_handoff.md and can_i2c_gateway_bom.csv"
+		(exclude_from_sim no)
+		(at 25.4 177.8 0)
+		(effects
+			(font
+				(size 1 1)
+				(italic yes)
+			)
+			(justify left bottom)
+		)
+	)
+(sheet_instances
     (path "/" (page "1"))
+      (path "/76314aad-fff2-4237-8c4a-2dbd4e06a2e1/762a1ab9-bdaa-41f1-9da1-1687126e729c" (page "2"))
+      (path "/76314aad-fff2-4237-8c4a-2dbd4e06a2e1/1f79907f-79dc-4a39-bb4a-b33268542400" (page "3"))
+      (path "/76314aad-fff2-4237-8c4a-2dbd4e06a2e1/ab8a1052-e2e8-4dde-ab61-e7465378221c" (page "4"))
+      (path "/76314aad-fff2-4237-8c4a-2dbd4e06a2e1/ca945800-30c4-4174-8f18-f8602dd80706" (page "5"))
   )
 )
