File: hardware/boards/backplane-backpack/01_power.kicad_sch (KiCad schematic)
At the start: 34 parts, among them J1 DC_IN, U4 LMR51610YDBVR, U5 LMR51610YDBVR

Commit message: chore: checkpoint current board layout
Other:
- moved on the sheet: C10, C11, C12, C13, C15, C17, C18, C20, C9, D2, L2, R19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

Commit message: hardware: mark all test points DNP
Parts:
- TP1, TP2, TP3, TP4: now not fitted; now left out of the parts list
Changed lines of the file:
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@@
 		(body_style 1)
 		(exclude_from_sim no)
-		(in_bom yes)
-		(on_board yes)
-		(in_pos_files yes)
-		(dnp no)
+		(in_bom no)
+		(on_board yes)
+		(in_pos_files yes)
+		(dnp yes)
 		(property "Reference" "TP1"
 			(at 35.56 87.884 0)
@@
 		(body_style 1)
 		(exclude_from_sim no)
-		(in_bom yes)
-		(on_board yes)
-		(in_pos_files yes)
-		(dnp no)
+		(in_bom no)
+		(on_board yes)
+		(in_pos_files yes)
+		(dnp yes)
 		(property "Reference" "TP2"
 			(at 38.354 108.204 0)
@@
 		(body_style 1)
 		(exclude_from_sim no)
-		(in_bom yes)
-		(on_board yes)
-		(in_pos_files yes)
-		(dnp no)
+		(in_bom no)
+		(on_board yes)
+		(in_pos_files yes)
+		(dnp yes)
 		(property "Reference" "TP3"
 			(at 37.592 100.076 0)
@@
 		(body_style 1)
 		(exclude_from_sim no)
-		(in_bom yes)
-		(on_board yes)
-		(in_pos_files yes)
-		(dnp no)
+		(in_bom no)
+		(on_board yes)
+		(in_pos_files yes)
+		(dnp yes)
 		(property "Reference" "TP4"
 			(at 39.624 118.618 0)
