File: hardware/boards/backplane-prototype/backplane-prototype.kicad_sch (KiCad schematic)
At the start: 32 parts, among them J1 SLOT_1, J2 i2c_backpack, J3 SLOT_2, J4 SLOT_3, J5 DC_IN, J6 SLOT_4, J7 SLOT_5, J8 SLOT_6

Commit message: Fix backplane connectivity and assembly metadata
Parts:
- H1, H2, H3, H4, H5, H6: footprint MountingHole:MountingHole_2.2mm_M2_Pad_Via -> mini-rack-power:MountingHole_2.2mm_M2_Pad_Via_JLC
- J1, J3, J4, J6, J7, J8: LCSC (none) -> C30170181; MPN (none) -> XT30U(2+2)-F.G.B; now not fitted
- J2: LCSC (none) -> C42391443; MPN (none) -> FG-PZ2.54-02-03P; now not fitted
- J5: now not fitted
Changed lines of the file:
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@@
 			)
 		)
-		(property "Footprint" "MountingHole:MountingHole_2.2mm_M2_Pad_Via"
+		(property "Footprint" "mini-rack-power:MountingHole_2.2mm_M2_Pad_Via_JLC"
 			(at 157.48 168.91 0)
 			(hide yes)
@@
 		(on_board yes)
 		(in_pos_files yes)
-		(dnp no)
+		(dnp yes)
 		(fields_autoplaced yes)
 		(property "Reference" "J8"
@@
 			)
 		)
+		(property "MPN" "XT30U(2+2)-F.G.B"
+			(at 223.52 45.72 0)
+			(hide yes)
+			(show_name no)
+			(do_not_autoplace no)
+			(effects
+				(font
+					(size 1.27 1.27)
+				)
+			)
+		)
+		(property "LCSC" "C30170181"
+			(at 223.52 45.72 0)
+			(hide yes)
+			(show_name no)
+			(do_not_autoplace no)
+			(effects
+				(font
+					(size 1.27 1.27)
+				)
+			)
+		)
 		(property "Pinout" "1=GND; 2=SLOT_6_PWR_SW; 3=SDA; 4=SCL"
 			(at 223.52 45.72 0)
@@
 			)
 		)
-		(property "Footprint" "MountingHole:MountingHole_2.2mm_M2_Pad_Via"
+		(property "Footprint" "mini-rack-power:MountingHole_2.2mm_M2_Pad_Via_JLC"
 			(at 142.24 168.91 0)
 			(hide yes)
@@
 			)
 		)
-		(property "Footprint" "MountingHole:MountingHole_2.2mm_M2_Pad_Via"
+		(property "Footprint" "mini-rack-power:MountingHole_2.2mm_M2_Pad_Via_JLC"
 			(at 129.54 168.91 0)
 			(hide yes)
@@
 		(on_board yes)
 		(in_pos_files yes)
-		(dnp no)
+		(dnp yes)
 		(fields_autoplaced yes)
 		(property "Reference" "J5"
@@
 			)
 		)
-		(property "Footprint" "MountingHole:MountingHole_2.2mm_M2_Pad_Via"
+		(property "Footprint" "mini-rack-power:MountingHole_2.2mm_M2_Pad_Via_JLC"
 			(at 142.24 182.88 0)
 			(hide yes)
@@
 			)
 		)
-		(property "Footprint" "MountingHole:MountingHole_2.2mm_M2_Pad_Via"
+		(property "Footprint" "mini-rack-power:MountingHole_2.2mm_M2_Pad_Via_JLC"
 			(at 157.48 182.88 0)
 			(hide yes)
@@
 		(on_board yes)
 		(in_pos_files yes)
-		(dnp no)
+		(dnp yes)
 		(fields_autoplaced yes)
 		(property "Reference" "J4"
@@
 			)
 		)
+		(property "MPN" "XT30U(2+2)-F.G.B"
+			(at 116.84 45.72 0)
+			(hide yes)
+			(show_name no)
+			(do_not_autoplace no)
+			(effects
+				(font
+					(size 1.27 1.27)
+				)
+			)
+		)
+		(property "LCSC" "C30170181"
+			(at 116.84 45.72 0)
+			(hide yes)
+			(show_name no)
+			(do_not_autoplace no)
+			(effects
+				(font
+					(size 1.27 1.27)
+				)
+			)
+		)
 		(property "Pinout" "1=GND; 2=SLOT_3_PWR_SW; 3=SDA; 4=SCL"
 			(at 116.84 45.72 0)
@@
 		(on_board yes)
 		(in_pos_files yes)
-		(dnp no)
+		(dnp yes)
 		(fields_autoplaced yes)
 		(property "Reference" "J1"
@@
 			)
 		)
+		(property "MPN" "XT30U(2+2)-F.G.B"
+			(at 45.72 45.72 0)
+			(hide yes)
+			(show_name no)
+			(do_not_autoplace no)
+			(effects
+				(font
+					(size 1.27 1.27)
+				)
+			)
+		)
+		(property "LCSC" "C30170181"
+			(at 45.72 45.72 0)
+			(hide yes)
+			(show_name no)
+			(do_not_autoplace no)
+			(effects
+				(font
+					(size 1.27 1.27)
+				)
+			)
+		)
 		(property "Pinout" "1=GND; 2=SLOT_1_PWR_SW; 3=SDA; 4=SCL"
 			(at 45.72 45.72 0)
@@
 		(on_board yes)
 		(in_pos_files yes)
-		(dnp no)
+		(dnp yes)
 		(fields_autoplaced yes)
 		(property "Reference" "J7"
@@
 			)
 		)
+		(property "MPN" "XT30U(2+2)-F.G.B"
+			(at 187.96 45.72 0)
+			(hide yes)
+			(show_name no)
+			(do_not_autoplace no)
+			(effects
+				(font
+					(size 1.27 1.27)
+				)
+			)
+		)
+		(property "LCSC" "C30170181"
+			(at 187.96 45.72 0)
+			(hide yes)
+			(show_name no)
+			(do_not_autoplace no)
+			(effects
+				(font
+					(size 1.27 1.27)
+				)
+			)
+		)
 		(property "Pinout" "1=GND; 2=SLOT_5_PWR_SW; 3=SDA; 4=SCL"
 			(at 187.96 45.72 0)
@@
 		(on_board yes)
 		(in_pos_files yes)
-		(dnp no)
+		(dnp yes)
 		(fields_autoplaced yes)
 		(property "Reference" "J2"
@@
 			)
 		)
+		(property "MPN" "FG-PZ2.54-02-03P"
+			(at 46.99 118.11 0)
+			(hide yes)
+			(show_name no)
+			(do_not_autoplace no)
+			(effects
+				(font
+					(size 1.27 1.27)
+				)
+			)
+		)
+		(property "LCSC" "C42391443"
+			(at 46.99 118.11 0)
+			(hide yes)
+			(show_name no)
+			(do_not_autoplace no)
+			(effects
+				(font
+					(size 1.27 1.27)
+				)
+			)
+		)
 		(pin "2"
 		)
@@
 		(on_board yes)
 		(in_pos_files yes)
-		(dnp no)
+		(dnp yes)
 		(fields_autoplaced yes)
 		(property "Reference" "J3"
@@
 			)
 		)
+		(property "MPN" "XT30U(2+2)-F.G.B"
+			(at 81.28 45.72 0)
+			(hide yes)
+			(show_name no)
+			(do_not_autoplace no)
+			(effects
+				(font
+					(size 1.27 1.27)
+				)
+			)
+		)
+		(property "LCSC" "C30170181"
+			(at 81.28 45.72 0)
+			(hide yes)
+			(show_name no)
+			(do_not_autoplace no)
+			(effects
+				(font
+					(size 1.27 1.27)
+				)
+			)
+		)
 		(property "Pinout" "1=GND; 2=SLOT_2_PWR_SW; 3=SDA; 4=SCL"
 			(at 81.28 45.72 0)
@@
 		(on_board yes)
 		(in_pos_files yes)
-		(dnp no)
+		(dnp yes)
 		(fields_autoplaced yes)
 		(property "Reference" "J6"
@@
 			)
 		)
+		(property "MPN" "XT30U(2+2)-F.G.B"
+			(at 152.4 45.72 0)
+			(hide yes)
+			(show_name no)
+			(do_not_autoplace no)
+			(effects
+				(font
+					(size 1.27 1.27)
+				)
+			)
+		)
+		(property "LCSC" "C30170181"
+			(at 152.4 45.72 0)
+			(hide yes)
+			(show_name no)
+			(do_not_autoplace no)
+			(effects
+				(font
+					(size 1.27 1.27)
+				)
+			)
+		)
 		(property "Pinout" "1=GND; 2=SLOT_4_PWR_SW; 3=SDA; 4=SCL"
 			(at 152.4 45.72 0)
@@
 			)
 		)
-		(property "Footprint" "MountingHole:MountingHole_2.2mm_M2_Pad_Via"
+		(property "Footprint" "mini-rack-power:MountingHole_2.2mm_M2_Pad_Via_JLC"
 			(at 129.54 182.88 0)
 			(hide yes)
