File: hardware/boards/backplane-prototype/05_buck_converters.kicad_sch (KiCad schematic)
At the start: 28 parts, among them U2 LM5164DDAR, U3 LM5164DDAR

Commit message: checkpoint: save fan and buck schematic edits
Other:
- note added: "VCC to +12V"
- note added: "VCC to +3v3"
- moved on the sheet: C10, C11, C12, C13, C9, L2, R10, R7, R8, R9, TP4

Commit message: Add second 3V3 buck output capacitor
Parts:
- added C14: 22uF 25V, Capacitor_SMD:C_0805_2012Metric, symbol Device:C
Connections:
- net +3V3: now also C14.1
- net GND: now also C14.2
Other:
- note added: "NOTES: - Both regulators are LM5164DDAR at approximately 300 kHz with 100 µH C2962892 inductors. - The +12 V rail follows TI's 12 V / 1 A Type-3 network except for the qualified 100 µH inductor. - +3V3 reuses the carrier's Type-3 values. - Input ceramics are rated for 100 V. - Each rail uses two 22 µF / 25 V output capacitors. TODO: - [ ] If the source is more than approximately 5 cm away, add or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"
Changed lines of the file:
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@@
 		)
 	)
-	(text_box "Both regulators are LM5164DDAR at approximately 300 kHz with 100 µH C2962892 inductors. The +12 V rail follows TI's 12 V / 1 A Type-3 network except for the qualified 100 µH inductor; +3V3 reuses the carrier's Type-3 values.\n\nInput ceramics are 100 V rated. Add or qualify bulk input capacitance during PCB layout if the source is more than approximately 5 cm away. Verify VIN ringing directly at each regulator, output ripple, PGOOD, inductor temperature, and fan startup/stall on first articles."
+	(text "NOTES:\n\n  - Both regulators are LM5164DDAR at approximately 300 kHz with 100 µH C2962892 inductors.\n  - The +12 V rail follows TI's 12 V / 1 A Type-3 network except for the qualified 100 µH inductor.\n  - +3V3 reuses the carrier's Type-3 values.\n  - Input ceramics are rated for 100 V.\n  - Each rail uses two 22 µF / 25 V output capacitors.\n\nTODO:\n\n  - [ ] If the source is more than approximately 5 cm away, add or qualify bulk input capacitance.\n  - [ ] On first articles, verify VIN ringing at each regulator, output ripple, PGOOD,\n        inductor temperature, and fan startup/stall.\n\nLAYOUT:\n\n  - Place input ceramics directly at each regulator's VIN/GND pins with a minimum-area loop.\n  - Place L1/L2 close to SW and minimize the SW copper area.\n  - Place C4/C14 at L1's output and C10/C11 at L2's output; return each pair directly to regulator GND/EP.\n  - Keep feedback and ripple-injection parts close to FB and away from SW."
 		(exclude_from_sim no)
-		(at 184.15 25.4 0)
-		(size 100.33 69.85)
-		(margins 1.27 1.27 1.27 1.27)
-		(stroke
-			(width 0)
-			(type solid)
-		)
-		(fill
-			(type none)
-		)
-		(effects
-			(font
-				(size 1.27 1.27)
-			)
-			(justify left top)
+		(at 184.15 81.28 0)
+		(effects
+			(font
+				(size 1.143 1.143)
+			)
+			(justify left bottom)
 		)
 	)
@@
 	(junction
 		(at 124.46 43.18)
+		(diameter 0)
+		(color 0 0 0 0)
+	)
+	(junction
+		(at 116.84 43.18)
 		(diameter 0)
 		(color 0 0 0 0)
@@
 		(pts
 			(xy 109.22 43.18) (xy 124.46 43.18)
+		)
+		(stroke
+			(width 0)
+			(type default)
+		)
+	)
+	(wire
+		(pts
+			(xy 109.22 50.8) (xy 116.84 50.8)
 		)
 		(stroke
@@
 		(dnp no)
 		(property "Reference" "C4"
-			(at 112.014 45.212 0)
-			(show_name no)
-			(do_not_autoplace no)
-			(effects
-				(font
-					(size 1.27 1.27)
-				)
-				(justify left)
+			(at 106.68 39.37 0)
+			(show_name no)
+			(do_not_autoplace no)
+			(effects
+				(font
+					(size 1.27 1.27)
+				)
+				(justify right)
 			)
 		)
 		(property "Value" "22uF 25V"
-			(at 112.014 47.498 0)
-			(show_name no)
-			(do_not_autoplace no)
-			(effects
-				(font
-					(size 1.27 1.27)
-				)
-				(justify left)
+			(at 106.68 36.83 0)
+			(show_name no)
+			(do_not_autoplace no)
+			(effects
+				(font
+					(size 1.27 1.27)
+				)
+				(justify right)
 			)
 		)
@@
 					(unit 1)
 				)
+			)
+		)
+	)
+	(symbol
+		(lib_id "Device:C")
+		(at 116.84 46.99 0)
+		(unit 1)
+		(body_style 1)
+		(exclude_from_sim no)
+		(in_bom yes)
+		(on_board yes)
+		(in_pos_files yes)
+		(dnp no)
+		(property "Reference" "C14"
+			(at 119.38 39.37 0)
+			(show_name no)
+			(do_not_autoplace no)
+			(effects
+				(font
+					(size 1.27 1.27)
+				)
+				(justify left)
+			)
+		)
+		(property "Value" "22uF 25V"
+			(at 119.38 36.83 0)
+			(show_name no)
+			(do_not_autoplace no)
+			(effects
+				(font
+					(size 1.27 1.27)
+				)
+				(justify left)
+			)
+		)
+		(property "Footprint" "Capacitor_SMD:C_0805_2012Metric"
+			(at 117.865 43.68 0)
+			(hide yes)
+			(show_name no)
+			(do_not_autoplace no)
+			(effects
+				(font
+					(size 1.27 1.27)
+				)
+			)
+		)
+		(property "Datasheet" ""
+			(at 116.9 47.49 0)
+			(hide yes)
+			(show_name no)
+			(do_not_autoplace no)
+			(effects
+				(font
+					(size 1.27 1.27)
+				)
+			)
+		)
+		(property "Description" ""
+			(at 116.9 47.49 0)
+			(hide yes)
+			(show_name no)
+			(do_not_autoplace no)
+			(effects
+				(font
+					(size 1.27 1.27)
+				)
+			)
+		)
+		(property "MPN" "CL21A226MAQNNNE"
+			(at 116.9 47.49 0)
+			(hide yes)
+			(show_name no)
+			(do_not_autoplace no)
+			(effects
+				(font
+					(size 1.27 1.27)
+				)
+			)
+		)
+		(property "Manufacturer" "Samsung Electro-Mechanics"
+			(at 116.9 47.49 0)
+			(hide yes)
+			(show_name no)
+			(do_not_autoplace no)
+			(effects
+				(font
+					(size 1.27 1.27)
+				)
+			)
+		)
+		(property "LCSC" "C45783"
+			(at 116.9 47.49 0)
+			(hide yes)
+			(show_name no)
+			(do_not_autoplace no)
+			(effects
+				(font
+					(size 1.27 1.27)
+				)
+			)
+		)
+		(property "Voltage" "25 V"
+			(at 116.9 47.49 0)
+			(hide yes)
+			(show_name no)
+			(do_not_autoplace no)
+			(effects
+				(font
+					(size 1.27 1.27)
+				)
+			)
+		)
+		(pin "1"
+		)
+		(pin "2"
+		)
+		(instances
+			(project "backplane-prototype"
+				(path "/348cc909-6345-4013-9bef-98714057a65b/9f6d14f1-eef5-43ec-a5a0-8ac65326e3cb"
+					(reference "C14")
+					(unit 1)
+				)

Commit message: checkpoint: save PCB schematic synchronization
Other:
- note added: "DC_IN/BUCK"
- note added: "NOTES: - Both regulators are LM5164DDAR at approximately 300 kHz with 100 µH inductors. - The +12 V rail follows TI's 12 V / 1 A Type-3 network except for the qualified 100 µH inductor. - +3V3 reuses carrier's schematic. - Input ceramics are rated for 100 V. - Each rail uses two 22 µF / 25 V output capacitors. TODO: - [ ] Verify VIN ringing at each regulator, output ripple, PGOOD inductor tempera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"
- note removed: "BUCK CONVERTERS: VCC TO +3V3 AND +12V"
- note removed: "NOTES: - Both regulators are LM5164DDAR at approximately 300 kHz with 100 µH C2962892 inductors. - The +12 V rail follows TI's 12 V / 1 A Type-3 network except for the qualified 100 µH inductor. - +3V3 reuses the carrier's Type-3 values. - Input ceramics are rated for 100 V. - Each rail uses two 22 µF / 25 V output capacitors. TODO: - [ ] If the source is more than approximately 5 cm away, add or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"
- moved on the sheet: C1, C10, C11, C12, C13, C14, C2, C3, C4, C5, C6, C7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
