File: hardware/boards/carrier/02_housekeeping.kicad_sch (KiCad schematic)
At the start: 10 parts, among them U1 STM32G031G6U6

Commit message: hardware: add carrier reset button
Parts:
- added SW1: SKSCLCE010, mini-rack-power:SW_ALPS_SKSCLCE010_SidePush, symbol Switch:SW_Push
- J2: now fitted
- LED1: value WS2812B-4020-V6 -> WS2812B-2020-V6; footprint mini-rack-power:LED_Worldsemi_WS2812B-4020_SideView -> LED_SMD:LED_WS2812B-2020_PLCC4_2.0x2.0mm; symbol mini-rack-power:WS2812B-4020-V6 -> LED:WS2812B-2020; Alternate_LCSC C52917434 -> (none); Alternate_MPN WS2812B-2020-V6 -> (none); LCSC C52941387 -> C52917434; MPN WS2812B-4020-V6 -> WS2812B-2020-V6; Population_Note Populate either the 4020 side-view pads or the 2020 top-emi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 -> (none)
Connections:
- net +3V3: now also LED1.4 (VDD); no longer LED1.2 (VDD)
- net GND: now also LED1.2 (VSS), SW1.1; no longer LED1.4 (VSS)
- net LED_DATA_RAW: now also LED1.3 (DIN); no longer LED1.1 (DIN)
- net NRST: now also SW1.2
Changed lines of the file:
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@@
 		(color 0 0 0 0)
+	)
+	(wire
+		(pts
+			(xy 20.32 50.8) (xy 20.32 55.88)
+		)
+		(stroke
+			(width 0)
+			(type default)
+		)
+	)
+	(wire
+		(pts
+			(xy 30.48 50.8) (xy 39.37 50.8)
+		)
+		(stroke
+			(width 0)
+			(type default)
+		)
 	)
 	(no_connect
@@
 		(in_bom yes)
 		(on_board yes)
-		(in_pos_files no)
-		(dnp yes)
+		(in_pos_files yes)
+		(dnp no)
 		(fields_autoplaced yes)
 		(property "Reference" "J2"
@@
 	)
 	(symbol
+		(lib_id "Switch:SW_Push")
+		(at 25.4 50.8 0)
+		(unit 1)
+		(body_style 1)
+		(exclude_from_sim no)
+		(in_bom yes)
+		(on_board yes)
+		(in_pos_files yes)
+		(dnp no)
+		(property "Reference" "SW1"
+			(at 25.4 47.498 0)
+			(show_name no)
+			(do_not_autoplace no)
+			(effects
+				(font
+					(size 1.27 1.27)
+				)
+			)
+		)
+		(property "Value" "SKSCLCE010"
+			(at 25.4 54.61 0)
+			(show_name no)
+			(do_not_autoplace no)
+			(effects
+				(font
+					(size 1.27 1.27)
+				)
+			)
+		)
+		(property "Footprint" "mini-rack-power:SW_ALPS_SKSCLCE010_SidePush"
+			(at 25.4 45.72 0)
+			(hide yes)
+			(show_name no)
+			(do_not_autoplace no)
+			(effects
+				(font
+					(size 1.27 1.27)
+				)
+			)
+		)
+		(property "Datasheet" "https://datasheet.lcsc.com/datasheet/pdf/a3d9c3c84b96b16ebda6f9dac2fc041f.pdf?productCode=C139799"
+			(at 25.4 50.8 0)
+			(hide yes)
+			(show_name no)
+			(do_not_autoplace no)
+			(effects
+				(font
+					(size 1.27 1.27)
+				)
+			)
+		)
+		(property "Description" "Low-profile right-angle side-push tactile switch, SPST-NO, 3.5 x 2.9 x 1.25 mm"
+			(at 25.4 50.8 0)
+			(hide yes)
+			(show_name no)
+			(do_not_autoplace no)
+			(effects
+				(font
+					(size 1.27 1.27)
+				)
+			)
+		)
+		(property "MPN" "SKSCLCE010"
+			(at 25.4 50.8 0)
+			(hide yes)
+			(show_name no)
+			(do_not_autoplace no)
+			(effects
+				(font
+					(size 1.27 1.27)
+				)
+			)
+		)
+		(property "Manufacturer" "ALPSALPINE"
+			(at 25.4 50.8 0)
+			(hide yes)
+			(show_name no)
+			(do_not_autoplace no)
+			(effects
+				(font
+					(size 1.27 1.27)
+				)
+			)
+		)
+		(property "LCSC" "C139799"
+			(at 25.4 50.8 0)
+			(hide yes)
+			(show_name no)
+			(do_not_autoplace no)
+			(effects
+				(font
+					(size 1.27 1.27)
+				)
+			)
+		)
+		(pin "1"
+		)
+		(pin "2"
+		)
+		(instances
+			(project "carrier"
+				(path "/ee42a069-09cc-4091-bee3-2dd6ab96c98c/64ed744c-f0e1-4d20-9137-f6a463447101"
+					(reference "SW1")
+					(unit 1)
+				)
+			)
+		)
+	)
+	(symbol
+		(lib_id "power:GND")
+		(at 20.32 55.88 0)
+		(unit 1)
+		(body_style 1)
+		(exclude_from_sim no)
+		(in_bom yes)
+		(on_board yes)
+		(in_pos_files yes)
+		(dnp no)
+		(fields_autoplaced yes)
+		(property "Reference" "#PWR68"
+			(at 20.32 62.23 0)
+			(hide yes)
+			(show_name no)
+			(do_not_autoplace no)
+			(effects
+				(font
+					(size 1.27 1.27)
+				)
+			)
+		)
+		(property "Value" "GND"
+			(at 20.32 60.96 0)
+			(show_name no)
+			(do_not_autoplace no)
+			(effects
+				(font
+					(size 1.27 1.27)
+				)
+			)
+		)
+		(property "Footprint" ""
+			(at 20.32 55.88 0)
+			(hide yes)
+			(show_name no)
+			(do_not_autoplace no)
+			(effects
+				(font
+					(size 1.27 1.27)
+				)
+			)
+		)
+		(property "Datasheet" ""
+			(at 20.32 55.88 0)
+			(hide yes)
+			(show_name no)
+			(do_not_autoplace no)
+			(effects
+				(font
+					(size 1.27 1.27)
+				)
+			)
+		)
+		(property "Description" "Power symbol creates a global label with name \"GND\" , ground"
+			(at 20.32 55.88 0)
+			(hide yes)
+			(show_name no)
+			(do_not_autoplace no)
+			(effects
+				(font
+					(size 1.27 1.27)
+				)
+			)
+		)
+		(pin "1"
+		)
+		(instances
+			(project "carrier"
+				(path "/ee42a069-09cc-4091-bee3-2dd6ab96c98c/64ed744c-f0e1-4d20-9137-f6a463447101"
+					(reference "#PWR68")
+					(unit 1)
+				)
+			)
+		)
+	)
+	(symbol
 		(lib_id "MCU_ST_STM32G0:STM32G031G6Ux")
 		(at 76.2 68.58 0)
@@
 	)
 	(symbol
-		(lib_id "mini-rack-power:WS2812B-4020-V6")
+		(lib_id "LED:WS2812B-2020")
 		(at 66.04 149.86 0)
 		(unit 1)
@@
 			)
 		)
-		(property "Value" "WS2812B-4020-V6"
+		(property "Value" "WS2812B-2020-V6"
 			(at 71.12 158.496 0)
 			(show_name no)
@@
 			)
 		)
-		(property "Footprint" "mini-rack-power:LED_Worldsemi_WS2812B-4020_SideView"
+		(property "Footprint" "LED_SMD:LED_WS2812B-2020_PLCC4_2.0x2.0mm"
 			(at 67.31 142.24 0)
 			(hide yes)
@@
 			)
 		)
-		(property "Datasheet" "https://datasheet.lcsc.com/datasheet/pdf/ec5ab06f6bef843823cdd508ed36b03e.pdf?productCode=C52941387"
+		(property "Datasheet" "https://cdn-shop.adafruit.com/product-files/4684/4684_WS2812B-2020_V1.3_EN.pdf"
 			(at 68.58 140.335 0)
 			(hide yes)
@@
 			)
 		)
-		(property "Description" "Side-view RGB LED with integrated WS2812-compatible controller, 3.3 V capable, 3.98 x 2.00 x 1.70 mm"
+		(property "Description" "RGB LED with integrated controller, 2.0 x 2.0 mm, 12 mA"
 			(at 66.04 149.86 0)
 			(hide yes)
@@
 			)
 		)
-		(property "MPN" "WS2812B-4020-V6"
+		(property "MPN" "WS2812B-2020-V6"
 			(at 66.04 149.86 0)
 			(hide yes)
@@
 			)
 		)
-		(property "LCSC" "C52941387"
+		(property "LCSC" "C52917434"
 			(at 66.04 149.86 0)
 			(hide yes)
-			(show_name no)
-			(do_not_autoplace no)
-			(effects
-				(font
-					(size 1.27 1.27)
-				)
-			)
-		)
-		(property "Alternate_MPN" "WS2812B-2020-V6"
-			(at 66.04 149.86 0)
-			(hide yes)
-			(show_name no)
-			(do_not_autoplace no)
-			(effects
-				(font
-					(size 1.27 1.27)
-				)
-			)
-		)
-		(property "Alternate_LCSC" "C52917434"
-			(at 66.04 149.86 0)
-			(hide yes)
-			(show_name no)
-			(do_not_autoplace no)
-			(effects
-				(font
-					(size 1.27 1.27)
-				)
-			)
-		)
-		(property "Population_Note" "Populate either the 4020 side-view pads or the 2020 top-emitting pads, never both"
-			(at 66.04 149.86 0)
-			(hide yes)
