File: hardware/boards/carrier/01_power_control.kicad_sch (KiCad schematic)
At the start: 42 parts, among them Q1 IPB020N10N5LF, Q2 2N7002, Q3 2N7002, U3 LMX5069MS, U4 INA237AIDGSR, U5 TCAN3413DR

Commit message: assign carrier LCSC assembly parts
Parts:
- C1: LCSC (none) -> C13832; MPN (none) -> CL31B105KCHNNNE; Manufacturer (none) -> Samsung Electro-Mechanics
- C10, C18: LCSC (none) -> C14663; MPN (none) -> CC0603KRX7R9BB104; Manufacturer (none) -> YAGEO
- C2: LCSC (none) -> C24797; MPN (none) -> 0603B684K160NT; Manufacturer (none) -> FH (Guangdong Fenghua Advanced Tech)
- R10: LCSC (none) -> C25803; MPN (none) -> 0603WAF1003T5E; Manufacturer (none) -> UNI-ROYAL (Uniroyal Elec)
- R11, R19: LCSC (none) -> C25804; MPN (none) -> 0603WAF1002T5E; Manufacturer (none) -> UNI-ROYAL (Uniroyal Elec)
- R17, R18: LCSC (none) -> C22859; MPN (none) -> 0603WAF100JT5E; Manufacturer (none) -> UNI-ROYAL (Uniroyal Elec)
- R2: LCSC (none) -> C22775; MPN (none) -> 0603WAF1000T5E; Manufacturer (none) -> UNI-ROYAL (Uniroyal Elec)
- R3, R9: LCSC (none) -> C23147; MPN (none) -> 0603WAF3602T5E; Manufacturer (none) -> UNI-ROYAL (Uniroyal Elec)
- R4, R6, R8: LCSC (none) -> C25805; MPN (none) -> 0603WAF1103T5E; Manufacturer (none) -> UNI-ROYAL (Uniroyal Elec)
- R5: LCSC (none) -> C25810; MPN (none) -> 0603WAF1802T5E; Manufacturer (none) -> UNI-ROYAL (Uniroyal Elec)
- R7: LCSC (none) -> C23186; MPN (none) -> 0603WAF5101T5E; Manufacturer (none) -> UNI-ROYAL (Uniroyal Elec)

Commit message: clean up carrier assembly BOM metadata
Parts:
- R3: value 36.0k 1% -> 36k 1%
Changed lines of the file:
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@@
 			)
 		)
-		(property "Value" "36.0k 1%"
+		(property "Value" "36k 1%"
 			(at 175.768 70.612 0)
 			(show_name no)

Commit message: consolidate carrier assembly parts
Parts:
- C15, C16: value 100nF 100V -> 100nF; LCSC C113803 -> C14663; MPN CC0603KRX7R0BB104 -> CC0603KRX7R9BB104; Manufacturer (none) -> YAGEO
Changed lines of the file:
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@@
 			)
 		)
-		(property "Value" "100nF 100V"
+		(property "Value" "100nF"
 			(at 130.81 224.536 0)
 			(show_name no)
@@
 			)
 		)
-		(property "MPN" "CC0603KRX7R0BB104"
+		(property "MPN" "CC0603KRX7R9BB104"
 			(at 129.54 222.25 0)
 			(hide yes)
@@
 			)
 		)
-		(property "LCSC" "C113803"
+		(property "Manufacturer" "YAGEO"
+			(at 129.54 222.25 0)
+			(hide yes)
+			(show_name no)
+			(do_not_autoplace no)
+			(effects
+				(font
+					(size 1.27 1.27)
+				)
+			)
+		)
+		(property "LCSC" "C14663"
 			(at 129.54 222.25 0)
 			(hide yes)
@@
 			)
 		)
-		(property "Value" "100nF 100V"
+		(property "Value" "100nF"
 			(at 147.066 224.79 0)
 			(show_name no)
@@
 			)
 		)
-		(property "MPN" "CC0603KRX7R0BB104"
+		(property "MPN" "CC0603KRX7R9BB104"
 			(at 146.05 222.25 0)
 			(hide yes)
@@
 			)
 		)
-		(property "LCSC" "C113803"
+		(property "Manufacturer" "YAGEO"
 			(at 146.05 222.25 0)
 			(hide yes)
+			(show_name no)
+			(do_not_autoplace no)
+			(effects
+				(font
+					(size 1.27 1.27)
+				)
+			)
+		)
+		(property "LCSC" "C14663"
+			(at 146.05 222.25 0)
+			(hide yes)

Commit message: clean carrier production routing and exports
Parts:
- TP17, TP18, TP19, TP20, TP21, TP22, TP23, TP24, TP25, TP26, TP6, TP7: now left out of the parts list
Changed lines of the file:
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@@
 		(body_style 1)
 		(exclude_from_sim no)
-		(in_bom yes)
+		(in_bom no)
 		(on_board yes)
-		(in_pos_files yes)
+		(in_pos_files no)
 		(dnp no)
 		(property "Reference" "TP23"
@@
 		(body_style 1)
 		(exclude_from_sim no)
-		(in_bom yes)
+		(in_bom no)
 		(on_board yes)
-		(in_pos_files yes)
+		(in_pos_files no)
 		(dnp no)
 		(property "Reference" "TP26"
@@
 		(body_style 1)
 		(exclude_from_sim no)
-		(in_bom yes)
+		(in_bom no)
 		(on_board yes)
-		(in_pos_files yes)
+		(in_pos_files no)
 		(dnp no)
 		(property "Reference" "TP17"
@@
 		(body_style 1)
 		(exclude_from_sim no)
-		(in_bom yes)
+		(in_bom no)
 		(on_board yes)
-		(in_pos_files yes)
+		(in_pos_files no)
 		(dnp no)
 		(property "Reference" "TP7"
@@
 		(body_style 1)
 		(exclude_from_sim no)
-		(in_bom yes)
+		(in_bom no)
 		(on_board yes)
-		(in_pos_files yes)
+		(in_pos_files no)
 		(dnp no)
 		(property "Reference" "TP21"
@@
 		(body_style 1)
 		(exclude_from_sim no)
-		(in_bom yes)
+		(in_bom no)
 		(on_board yes)
-		(in_pos_files yes)
+		(in_pos_files no)
 		(dnp no)
 		(property "Reference" "TP6"
@@
 		(body_style 1)
 		(exclude_from_sim no)
-		(in_bom yes)
+		(in_bom no)
 		(on_board yes)
-		(in_pos_files yes)
+		(in_pos_files no)
 		(dnp no)
 		(property "Reference" "TP18"
@@
 		(body_style 1)
 		(exclude_from_sim no)
-		(in_bom yes)
+		(in_bom no)
 		(on_board yes)
-		(in_pos_files yes)
+		(in_pos_files no)
 		(dnp no)
 		(property "Reference" "TP20"
@@
 		(body_style 1)
 		(exclude_from_sim no)
-		(in_bom yes)
+		(in_bom no)
 		(on_board yes)
-		(in_pos_files yes)
+		(in_pos_files no)
 		(dnp no)
 		(property "Reference" "TP25"
@@
 		(body_style 1)
 		(exclude_from_sim no)
-		(in_bom yes)
+		(in_bom no)
 		(on_board yes)
-		(in_pos_files yes)
+		(in_pos_files no)
 		(dnp no)
 		(property "Reference" "TP19"
@@
 		(body_style 1)
 		(exclude_from_sim no)
-		(in_bom yes)
+		(in_bom no)
 		(on_board yes)
-		(in_pos_files yes)
+		(in_pos_files no)
 		(dnp no)
 		(property "Reference" "TP24"
@@
 		(body_style 1)
 		(exclude_from_sim no)
-		(in_bom yes)
+		(in_bom no)
 		(on_board yes)
-		(in_pos_files yes)
+		(in_pos_files no)
 		(dnp no)
 		(property "Reference" "TP22"

Commit message: document carrier validation and datasheet set
Other:
- note added: "CAN PLACEMENT: keep D2, L3, and U5 close to J1 (connector → D2 → L3 → U5). D2 is at the closest location that clears J1 and preserves post-assembly soldering access; keep its remaining CAN stubs and ground connection short. Place C15/C16 directly at U5 VCC/VIO. Route CAN_BUS_P/N and CAN_PHY_P/N as differential pairs; P = CANH, N = CANL. Keep each pair short, tightly coupled, symmetric, and length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"
- note removed: "CAN PLACEMENT: keep D2, L3, and U5 close to J1 (connector → D2 → L3 → U5). Place C15/C16 directly at U5 VCC/VIO. Route CAN_BUS_P/N and CAN_PHY_P/N as differential pairs; P = CANH, N = CANL. Keep each pair short, tightly coupled, symmetric, and length-matched. Route CAN_TX/CAN_RX over continuous ground, away from switching nodes. J1 is fixed: preserve physical N/P pair order through D2 and L3; L3 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"
Changed lines of the file:
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@@
 		)
 	)
-	(text "CAN PLACEMENT: keep D2, L3, and U5 close to J1 (connector → D2 → L3 → U5).\nPlace C15/C16 directly at U5 VCC/VIO. Route CAN_BUS_P/N and CAN_PHY_P/N as differential pairs; P = CANH, N = CANL.\nKeep each pair short, tightly coupled, symmetric, and length-matched. Route CAN_TX/CAN_RX over continuous ground, away from switching nodes.\nJ1 is fixed: preserve physical N/P pair order through D2 and L3; L3 pads 1/4 = N and pads 2/3 = P."
+	(text "CAN PLACEMENT: keep D2, L3, and U5 close to J1 (connector → D2 → L3 → U5).\nD2 is at the closest location that clears J1 and preserves post-assembly soldering access; keep its remaining CAN stubs and ground connection short.\nPlace C15/C16 directly at U5 VCC/VIO. Route CAN_BUS_P/N and CAN_PHY_P/N as differential pairs; P = CANH, N = CANL.\nKeep each pair short, tightly coupled, symmetric, and length-matched. Route CAN_TX/CAN_RX over continuous ground, away from switching nodes.\nJ1 is fixed: preserve physical N/P pair order through D2 and L3; L3 pads 1/4 = N and pads 2/3 = P."
 		(exclude_from_sim no)
 		(at 23.876 221.742 0)

Commit message: use no-fee SMCJ48A assembly alternate
Parts:
- D1: LCSC C5861043 -> C19077611; Manufacturer (none) -> Zhuhai Hongjiacheng Technology
Changed lines of the file:
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@@
 			)
 		)
-		(property "Datasheet" ""
+		(property "Datasheet" "https://wmsc.lcsc.com/wmsc/upload/file/pdf/v2/lcsc/2312280929_hongjiacheng-SMCJ48A_C19077611.pdf"
 			(at 29.21 44.45 0)
 			(hide yes)
@@
 			)
 		)
-		(property "Description" "Zener diode"
+		(property "Description" "1500 W unidirectional 48 V TVS diode, SMC (DO-214AB)"
 			(at 29.21 44.45 0)
 			(hide yes)
@@
 			)
 		)
-		(property "LCSC" "C5861043"
+		(property "Manufacturer" "Zhuhai Hongjiacheng Technology"
 			(at 29.21 44.45 0)
 			(hide yes)
+			(show_name no)
+			(do_not_autoplace no)
+			(effects
+				(font
+					(size 1.27 1.27)
+				)
+			)
+		)
+		(property "LCSC" "C19077611"
+			(at 29.21 44.45 0)
+			(hide yes)

Commit message: hardware: mark all test points DNP
Parts:
- TP17, TP18, TP19, TP20, TP21, TP22, TP23, TP24, TP25, TP26, TP6, TP7: now not fitted
Changed lines of the file:
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@@
 		(on_board yes)
 		(in_pos_files no)
-		(dnp no)
+		(dnp yes)
 		(property "Reference" "TP23"
 			(at 68.58 140.208 0)
@@
 		(on_board yes)
 		(in_pos_files no)
-		(dnp no)
+		(dnp yes)
 		(property "Reference" "TP26"
 			(at 144.78 119.888 0)
@@
 		(on_board yes)
 		(in_pos_files no)
-		(dnp no)
+		(dnp yes)
 		(property "Reference" "TP17"
 			(at 55.88 240.538 0)
@@
 		(on_board yes)
 		(in_pos_files no)
-		(dnp no)
+		(dnp yes)
 		(property "Reference" "TP7"
 			(at 116.078 237.744 0)
@@
 		(on_board yes)
 		(in_pos_files no)
-		(dnp no)
+		(dnp yes)
 		(property "Reference" "TP21"
 			(at 106.68 119.888 0)
@@
 		(on_board yes)
 		(in_pos_files no)
-		(dnp no)
+		(dnp yes)
 		(property "Reference" "TP6"
 			(at 115.824 245.872 0)
@@
 		(on_board yes)
 		(in_pos_files no)
-		(dnp no)
+		(dnp yes)
 		(property "Reference" "TP18"
 			(at 55.88 249.174 0)
@@
 		(on_board yes)
 		(in_pos_files no)
-		(dnp no)
+		(dnp yes)
 		(property "Reference" "TP20"
 			(at 68.58 119.888 0)
@@
 		(on_board yes)
 		(in_pos_files no)
-		(dnp no)
+		(dnp yes)
 		(property "Reference" "TP25"
 			(at 144.78 140.208 0)
@@
 		(on_board yes)
 		(in_pos_files no)
-		(dnp no)
+		(dnp yes)
 		(property "Reference" "TP19"
 			(at 30.48 119.888 0)
@@
 		(on_board yes)
 		(in_pos_files no)
-		(dnp no)
+		(dnp yes)
 		(property "Reference" "TP24"
 			(at 106.68 140.208 0)
@@
 		(on_board yes)
 		(in_pos_files no)
-		(dnp no)
+		(dnp yes)
 		(property "Reference" "TP22"
 			(at 30.48 140.208 0)
